File: green-shield-hardware/green-shield-hardware.sch (KiCad schematic (older format))
At the start: 30 parts, among them J1 Conn_01x06_Female, J2 Conn_01x06_Female, J3 Conn_01x10_Female, J4 Conn_01x08_Female, J5 TB3, J6 TB3, J7 TB1, J8 TB2, U1 LM358, U2 LM358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

Commit message: finish pcb layout
Parts:
- removed J1, J2: Conn_01x06_Female, symbol Connector:Conn_01x06_Female
- removed J3: Conn_01x10_Female, symbol Connector:Conn_01x10_Female
- removed J4: Conn_01x08_Female, symbol Connector:Conn_01x08_Female
- removed U2: LM358, symbol Amplifier_Operational:LM358
- added D5, D6: LED, LED_SMD:LED_0603_1608Metric, symbol Device:LED
- added J1, J2: Conn_01x06_Male, Connector_PinSocket_2.54mm:PinSocket_1x06_P2.54mm_Vertical, symbol Connector:Conn_01x06_Male
- added J3: Conn_01x10_Male, Connector_PinSocket_2.54mm:PinSocket_1x10_P2.54mm_Vertical, symbol Connector:Conn_01x10_Male
- added J4: Conn_01x08_Male, Connector_PinSocket_2.54mm:PinSocket_1x08_P2.54mm_Vertical, symbol Connector:Conn_01x08_Male
- added R13, R14: 1K, Resistor_SMD:R_0603_1608Metric, symbol Device:R_Small
- added unit 2 of U1
- D1, D2, D3, D4: footprint (none) -> LED_SMD:LED_0603_1608Metric
- J5: footprint (none) -> TerminalBlock:TerminalBlock_Altech_AK300-2_P5.00mm
- J6: value TB3 -> TB4; footprint (none) -> TerminalBlock:TerminalBlock_Altech_AK300-2_P5.00mm
- J7, J8: footprint (none) -> TerminalBlock:TerminalBlock_Altech_AK300-3_P5.00mm
- R1, R10, R2, R3, R4, R5, R6, R7, R8, R9: footprint (none) -> Resistor_SMD:R_0603_1608Metric
- R11, R12: footprint (none) -> Relay_THT:Relay_SPDT_SANYOU_SRD_Series_Form_C
- RV1, RV2: footprint (none) -> Potentiometer_THT:Potentiometer_ACP_CA9-V10_Vertical_Hole
- U1: footprint (none) -> Package_TO_SOT_SMD:SOT-23-8
- U3: footprint (none) -> Package_DIP:DIP-16_W7.62mm_Socket
Connections:
- net +5V: now also J1.4 (Pin_4)
- net A0: now also J2.6 (Pin_6)
- net A1: now also J2.5 (Pin_5), U1.7
- net D2: now also J4.6 (Pin_6)
- net D3: now also J4.5 (Pin_5)
- net D4: now also J4.4 (Pin_4)
- net D5: now also J4.3 (Pin_3)
- net D6: now also J4.2 (Pin_2)
- net D7: now also J4.1 (Pin_1)
- net D8: now also J3.10 (Pin_10)
- net GND: now also J1.2 (Pin_2), J1.3 (Pin_3), J3.4 (Pin_4), R13.2, R14.2
- net at R12.4 (VCC), U3.12 (O5): now also D6.1 (K)
- net at R11.4 (VCC), U3.11 (O6): now also D5.1 (K)
- net at J6.1 (Pin_1), R2.1, R4.1: now also U1.6 (-)
- net at RV2.3: now also U1.5 (+)
- new net: D6.2 (A), R14.1
- new net: D5.2 (A), R13.1
